Commit message: 去除了base footprint 试图增加mecanum driver

File: src/sentry_simulation/urdf/imu.urdf.xacro (robot description, xacro)
@@ -3,5 +3,5 @@
     <xacro:property name="update_rate" value="100" />
     <xacro:property name="visualize" value="true" />
-    <xacro:property name="imu_topic" value="imu" />
+    <xacro:property name="imu_topic" value="/livox/imu" />
     <xacro:property name="body_name" value="imu_link" />
     <xacro:property name="update_RateHZ" value="100.0" />
@@ -25,5 +25,10 @@
             <material name="Red" />
         </collision>
-        <xacro:inertial_matrix mass="0.05" />
+        <inertial>
+            <mass value="1e-2" />
+            <origin xyz="0 0 0" rpy="0 0 0" />
+            <inertia ixx="1e-6" ixy="0.0" ixz="0"
+                     iyy="0.0"  iyz="0.0" izz="1e-6" />
+        </inertial>
     </link>
     <joint name="imu_joint" type="fixed">

File: src/sentry_simulation/urdf/livox_mid360.urdf.xacro (robot description, xacro)
@@ -13,5 +13,5 @@
   <xacro:property name="samples" value="20000" />
   <xacro:property name="downsample" value="1" />
-  <xacro:property name="ros_topic" value="livox_horizon_points" />
+  <xacro:property name="ros_topic" value="/livox/lidar" />
   <!-- Macro for inertia matrix -->
   <xacro:macro name="sphere_inertial_matrix" params="m r">
@@ -89,5 +89,5 @@
       <visualize>${visualize}</visualize>
       <update_rate>${update_rate}</update_rate>
-        <!-- This ray plugin is only for visualization. -->
+      <!-- This ray plugin is only for visualization. -->
       <plugin name="gazebo_ros_laser_controller" filename="libsentry_simulation.so">
         <ray>

File: src/sentry_simulation/urdf/sentry_base.urdf.xacro (robot description, xacro)
@@ -13,4 +13,7 @@
         <color rgba="1 0 0 1" />
     </material>
+    <material name="Green">
+        <color rgba="0 1 0 1" />
+    </material>
     <material name="Brown">
         <color rgba="0.647 0.165 0.165 1" />
@@ -19,5 +22,5 @@
 	<xacro:property name="length_wheel" value="0.05" />
 	<xacro:property name="radius_wheel" value="0.06" />
-    <xacro:property name="mass_wheel" value="150" />
+    <xacro:property name="mass_wheel" value="50" />
     <xacro:property name="mass_baselink" value="250" />
     <!-- Inertial matrix  -->
@@ -26,6 +29,6 @@
             <mass value="${mass}" />
             <origin xyz="0 0 0" rpy="0 0 0" />
-            <inertia ixx="2.3319" ixy="3.6592E-17" ixz="-4.7325E-18"
-                     iyy="2.4738" iyz="-2.8587E-19" izz="4.7802" />
+            <inertia ixx="2.3319" ixy="0.0" ixz="0.0"
+                     iyy="2.4738" iyz="0.0" izz="4.7802" />
         </inertial>
     </xacro:macro>
@@ -38,20 +41,4 @@
     <!-- //////////////////////////////// all base links of sentry ////////////////////////////////// -->
     <link name="dummy" />
-    <link name="base_footprint">
-        <visual>
-            <origin xyz="0 0 0" rpy="0 0 0" />
-            <geometry>
-                <box size="0.001 0.001 0.001" />
-            </geometry>
-            <material name="Blue" />
-        </visual>
-        <collision>
-            <origin xyz="0 0 0" rpy="0 0 0" />
-            <geometry>
-                <box size="0.1 0.1 0.1" />
-            </geometry>
-        </collision>
-        <xacro:inertial_matrix mass="0.000001"/>
-    </link>
     <link name="base_link">
         <visual>
@@ -138,11 +125,6 @@
         <origin xyz="0 0 0" />
         <parent link="dummy" />
-        <child link="base_footprint" />
+        <child link="base_link" />
     </joint>
-	<joint name="base_footprint_joint" type="fixed">
-		<origin xyz="0 0 0" />
-		<parent link="base_footprint" />
-		<child link="base_link" />
-	</joint>
     <joint name="base_to_wheel1" type="continuous">
         <axis xyz="0 0 1" />
@@ -178,5 +160,4 @@
     </joint>
     <!-- //////////////////////////////// gazebo ////////////////////////////////// -->
-    <xacro:gazebo_material ref="base_footprint"    color="White" />
     <xacro:gazebo_material ref="base_link"         color="Orange" />
     <xacro:gazebo_material ref="left_front_wheel"  color="Black" />
@@ -184,25 +165,16 @@
     <xacro:gazebo_material ref="left_rear_wheel"   color="Red" />
     <xacro:gazebo_material ref="right_rear_wheel"  color="Red" />
-    <!-- //// ////////////////////////////// driver controller //////////////////////////////////  -->
+    <!-- //// ////////////////////////////// driver controller ///////////////////  -->
     <gazebo>
         <plugin name="mecanum_controller" filename="libgazebo_ros_planar_move.so">
-            <always_on>true</always_on>
-            <updateRate>100.0</updateRate>
             <robotNamespace>/</robotNamespace>
             <commandTopic>cmd_vel</commandTopic>
             <odometryTopic>odom</odometryTopic>
             <odometryFrame>odom</odometryFrame>
-            <leftFrontJoint>base_to_wheel1</leftFrontJoint>
-            <rightFrontJoint>base_to_wheel3</rightFrontJoint>
-            <leftRearJoint>base_to_wheel2</leftRearJoint>
-            <rightRearJoint>base_to_wheel4</rightRearJoint>
-            <wheelSeparation>0.26</wheelSeparation>
-            <wheelDiameter>0.12</wheelDiameter>
             <odometryRate>20.0</odometryRate>
-            <torque>2</torque>
-            <robotBaseFrame>base_footprint</robotBaseFrame>
+            <robotBaseFrame>base_link</robotBaseFrame>
+            <cmdTimeout>3.0</cmdTimeout>
             <publishOdomTF>false</publishOdomTF>
             <broadcastTF>false</broadcastTF>
-            <cmdTimeout>3.0</cmdTimeout>
         </plugin>
     </gazebo>

Commit message: 将初始位姿和relocation结合

File: src/sentry_simulation/urdf/imu.urdf.xacro (robot description, xacro)
@@ -36,5 +36,5 @@
         <parent link="base_link" />
         <child link="imu_link" />
-        <origin xyz="0.125  0 0.2" rpy="${PI} 0 0" />
+        <origin xyz="0.125  0 0.2" rpy="0 0 0" />
     </joint>
     <!-- //////////////////////////////// imu control ////////////////////////////////// -->

File: src/sentry_simulation/urdf/livox_mid360.urdf.xacro (robot description, xacro)
@@ -80,5 +80,5 @@
   </link>
   <joint name="livox_mid360_platform" type="fixed">
-    <origin xyz="0.05 0 -0.05" rpy="${PI} 0 0" />
+    <origin xyz="0.05 0 -0.05" rpy="0 0 0" />
     <parent link="livox_platform" />
     <child link="livox_mid360" />
