Commit message: 优化了simulation代码结构

File: src/sentry_simulation/urdf/sentry.urdf.xacro (robot description, xacro)
@@ -1,3 +1,3 @@
-<robot name="sentry_base" xmlns:xacro="http://www.ros.org/wiki/xacro">
+<robot name="sentry" xmlns:xacro="http://www.ros.org/wiki/xacro">
     <!-- Defining the colors used in this robot  -->
     <material name="Black">
@@ -28,5 +28,4 @@
     <xacro:property name="update_rate" value="100" />
     <xacro:property name="visualize" value="true" />
-    <xacro:property name="imu_topic" value="/livox/imu" />
     <xacro:property name="body_name" value="imu_link" />
     <xacro:property name="update_RateHZ" value="100.0" />
@@ -35,4 +34,5 @@
     <xacro:property name="queueSize" value="100" />
     <xacro:property name="PI" value="3.1415926"/>
+    <xacro:property name="imu_topic" value="/livox/imu" />
     <!-- //////////////////////////////// lidar ////////////////////////////////// -->
     <xacro:property name="visualize" value="true" />
@@ -237,9 +237,9 @@
             <odometryTopic>odom</odometryTopic>
             <odometryFrame>odom</odometryFrame>
-            <odometryRate>20.0</odometryRate>
+            <odometryRate>10.0</odometryRate>
             <robotBaseFrame>base_link</robotBaseFrame>
             <cmdTimeout>3.0</cmdTimeout>
-            <publishOdomTF>false</publishOdomTF>
-            <broadcastTF>false</broadcastTF>
+            <publishOdomTF>False</publishOdomTF>
+            <broadcastTF>False</broadcastTF>
         </plugin>
     </gazebo>
@@ -268,45 +268,44 @@
     </gazebo>
     <!-- //////////////////////////////// lidar control ////////////////////////////////// -->
-    <!-- 16线120度雷达  -->
     <gazebo reference="livox_mid360">
-        <sensor type="ray" name="livox_frame">
+      <sensor type="ray" name="livox_mid360">
         <pose>0 0 0 0 0 0</pose>
-        <visualize>false</visualize>
-        <visualize>true</visualize>
-        <update_rate>10</update_rate>
-        <ray>
-            <scan>
-            <horizontal>
-                <samples>1800</samples>
-                <resolution>0.2</resolution>
-                <min_angle>-3.14</min_angle>
-                <max_angle>3.14</max_angle>
-            </horizontal>
-            <vertical>
-                <samples>16</samples>
-                <resolution>2</resolution>
-                <min_angle>-0.2616</min_angle>
-                <max_angle> 0.2616</max_angle>
-            </vertical>
-        </scan>
-        <range>
-          <min>1</min>
-          <max>100.0</max>
-          <resolution>0.1</resolution>
-        </range>
-        <noise>
-          <type>gaussian</type>
-          <mean>0.0</mean>
-          <stddev>0.0</stddev>
-        </noise>
-      </ray>
-      <plugin name="gazebo_ros_laser_controller" filename="libgazebo_ros_velodyne_laser.so">
-        <topicName>/livox/lidar</topicName>
-        <frameName>livox_mid360</frameName>
-         <min_range>0.9</min_range>
-          <max_range>130.0</max_range>
-          <gaussianNoise>0.0</gaussianNoise>
-      </plugin>
-    </sensor>
-  </gazebo>
+        <visualize>${visualize}</visualize>
+        <update_rate>${update_rate}</update_rate>
+        <!-- This ray plugin is only for visualization. -->
+        <plugin name="gazebo_ros_laser_controller" filename="libsentry_simulation.so">
+            <ray>
+                <scan>
+                  <horizontal>
+                    <samples>0</samples>
+                    <resolution>1</resolution>
+                    <min_angle>${0}</min_angle>
+                    <max_angle>${2*PI}</max_angle>
+                  </horizontal>
+                  <vertical>
+                    <samples>0</samples>
+                    <resolution>1</resolution>
+                    <min_angle>${-7.22/180*PI}</min_angle>
+                    <max_angle>${55.22/180*PI}</max_angle>
+                  </vertical>
+                </scan>
+                <range>
+                  <min>${laser_min_range}</min>
+                  <max>${laser_max_range}</max>
+                  <resolution>${resolution}</resolution>
+                </range>
+                <noise>
+                  <type>gaussian</type>
+                  <mean>${noise_mean}</mean>
+                  <stddev>${noise_stddev}</stddev>
+                </noise>
+            </ray>
+            <samples>${samples}</samples>
+    	    <downsample>${downsample}</downsample>
+    	    <csv_file_name>package://sentry_simulation/scan_mode/mid360.csv</csv_file_name>
+    	    <ros_topic>${ros_topic}</ros_topic>
+            <broadcastTF>false</broadcastTF>
+        </plugin>
+      </sensor>
+    </gazebo>
 </robot>
