Commit message: run with old model

File: src/sentry_simulation/urdf/sentry_acker.urdf.xacro (robot description, xacro)
@@ -199,7 +199,7 @@
     </joint>
     <joint name="base_lidar" type="fixed">
-        <origin xyz="0.135 0 0.23" rpy="0 0 3.1415926" />
         <parent link="base_link" />
         <child link="livox_mid360" />
+        <origin xyz="0.135 0 0.23" rpy="0 0 0" />
     </joint>
     <!-- //////////////////////////////// gazebo ////////////////////////////////// -->
@@ -216,5 +216,5 @@
             <!-- 因为关闭发布odom的tf没有效果，所以此处把parent link改为gazebo_odom,child link改为gazebo_base_link
             仍可以通过cmd_vel话题来控制小车的运动，同时可以跑其他里程计算法，避免干扰 -->
-            <odometryTopic>odom</odometryTopic>
+            <odometryTopic>/gazebo_odom</odometryTopic>
             <odometryRate>10.0</odometryRate>
             <odometryFrame>gazebo_odom</odometryFrame>
@@ -252,5 +252,5 @@
       <sensor type="ray" name="livox_mid360">
         <pose>0 0 0 0 0 0</pose>
-        <visualize>false</visualize>
+        <visualize>true</visualize>
         <update_rate>10</update_rate>
         <!-- This ray plugin is only for visualization. -->
@@ -282,5 +282,5 @@
                 </noise>
             </ray>
-            <visualize>True</visualize>
+            <visualize>false</visualize>
             <samples>20000</samples>
     	    <downsample>1</downsample>
