Commit message: change the model of mid360

File: src/sentry_simulation/urdf/main.urdf.xacro (robot description, xacro)
@@ -2,35 +2,29 @@
 <robot xmlns:xacro="http://www.ros.org/wiki/xacro" name="open_base">
 	<xacro:include filename="$(find sentry_simulation)/urdf/rim.urdf.xacro"/>
-	<link name="origin_link"/>
 	<link name="base_link">
-	<inertial>
-		<mass value="0.07862944645"/>
-		<inertia
-			ixx="0.00002035985530754"
-			ixy="0"
-			ixz="0"
-			iyy="0.00002035985530754"
-			iyz="0"
-			izz="0.00003945961663220"/>
-		</inertial>
-	<visual>
-		<geometry>
-			<mesh filename="package://sentry_simulation/mesh/omni/base.stl"/>
-		</geometry>
-		<material name="base_material">
-			<color rgba="1 1 1 1"/>
-		</material>
-	</visual>
-	<collision>
-		<geometry>
-			<mesh filename="package://sentry_simulation/mesh/omni/base.stl"/>
-		</geometry>
-	</collision>
+		<inertial>
+			<mass value="0.07862944645"/>
+			<inertia
+				ixx="0.00002035985530754"
+				ixy="0"
+				ixz="0"
+				iyy="0.00002035985530754"
+				iyz="0"
+				izz="0.00003945961663220"/>
+			</inertial>
+		<visual>
+			<geometry>
+				<mesh filename="package://sentry_simulation/mesh/omni/base.stl"/>
+			</geometry>
+			<material name="base_material">
+				<color rgba="1 1 1 1"/>
+			</material>
+		</visual>
+		<collision>
+			<geometry>
+				<mesh filename="package://sentry_simulation/mesh/omni/base.stl"/>
+			</geometry>
+		</collision>
 	</link>
-	<joint name="base_joint" type="fixed">
-		<parent link="origin_link" />
-		<child link="base_link" />
-		<origin xyz="0 0 0.01905"/>
-	</joint>
 	<xacro:rim_macro
 		name="front_left"

File: src/sentry_simulation/urdf/sentry_acker.urdf.xacro (robot description, xacro)
@@ -25,25 +25,4 @@
     <xacro:property name="mass_baselink" value="250" />
     <!-- //////////////////////////////// imu ////////////////////////////////// -->
-    <xacro:property name="always_on" value="true" />
-    <xacro:property name="update_rate" value="100" />
-    <xacro:property name="visualize" value="true" />
-    <xacro:property name="body_name" value="imu_link" />
-    <xacro:property name="update_RateHZ" value="100.0" />
-    <xacro:property name="gaussian_noise" value="0.0" />
-    <xacro:property name="frame_name" value="imu_link" />
-    <xacro:property name="queueSize" value="100" />
-    <xacro:property name="PI" value="3.1415926"/>
-    <xacro:property name="imu_topic" value="/livox/imu" />
-    <!-- //////////////////////////////// lidar ////////////////////////////////// -->
-    <xacro:property name="visualize" value="true" />
-    <xacro:property name="update_rate" value="10" />
-    <xacro:property name="resolution" value="0.002" />
-    <xacro:property name="laser_min_range" value="0.1" />
-    <xacro:property name="laser_max_range" value="200.0" />
-    <xacro:property name="noise_mean" value="0.00" />
-    <xacro:property name="noise_stddev" value="0.00" />
-    <xacro:property name="samples" value="20000" />
-    <xacro:property name="downsample" value="1" />
-    <xacro:property name="ros_topic" value="/livox/lidar" />
     <!-- Inertial matrix  -->
     <xacro:macro name="inertial_matrix" params="mass">
@@ -168,5 +147,5 @@
             <origin xyz="0 0 0" rpy="0 0 0" />
             <geometry>
-                <mesh filename="package://sentry_simulation/mesh/livox_mid360.dae">
+                <mesh filename="package://sentry_simulation/mesh/mid360.stl">
                 </mesh>
             </geometry>
@@ -175,5 +154,5 @@
             <origin xyz="0 0 0" rpy="0 0 0" />
             <geometry>
-                <mesh filename="package://sentry_simulation/mesh/livox_mid360.dae">
+                <mesh filename="package://sentry_simulation/mesh/mid360.stl">
                 </mesh>
             </geometry>
@@ -220,5 +199,5 @@
     </joint>
     <joint name="base_lidar" type="fixed">
-        <origin xyz="0.175 0 0.46" rpy="0 0 0" />
+        <origin xyz="0.135 0 0.23" rpy="0 0 3.1415926" />
         <parent link="base_link" />
         <child link="livox_mid360" />
@@ -235,8 +214,10 @@
             <robotNamespace>/</robotNamespace>
             <commandTopic>cmd_vel</commandTopic>
+            <!-- 因为关闭发布odom的tf没有效果，所以此处把parent link改为gazebo_odom,child link改为gazebo_base_link
+            仍可以通过cmd_vel话题来控制小车的运动，同时可以跑其他里程计算法，避免干扰 -->
             <odometryTopic>odom</odometryTopic>
-            <odometryFrame>odom</odometryFrame>
             <odometryRate>10.0</odometryRate>
-            <robotBaseFrame>base_link</robotBaseFrame>
+            <odometryFrame>gazebo_odom</odometryFrame>
+            <robotBaseFrame>gazebo_base_link</robotBaseFrame>
             <cmdTimeout>3.0</cmdTimeout>
             <publishOdomTF>False</publishOdomTF>
@@ -250,17 +231,17 @@
         <gravity>true</gravity>
         <sensor name="imu_sensor" type="imu">
-            <always_on>${always_on}</always_on>
-            <update_rate>${update_rate}</update_rate>
-            <visualize>${visualize}</visualize>
+            <always_on>true</always_on>
+            <update_rate>100</update_rate>
+            <visualize>true</visualize>
             <topic>_default_topic_</topic>
             <plugin filename="libgazebo_ros_imu_sensor.so" name="imu_plugin">
-                <topicName>${imu_topic}</topicName>
-                <bodyName>${body_name}</bodyName>
-                <updateRateHZ>${update_RateHZ}</updateRateHZ>
-                <gaussianNoise>${gaussian_noise}</gaussianNoise>
-                <frameName>${frame_name}</frameName>
+                <topicName>/livox/imu</topicName>
+                <bodyName>imu_link</bodyName>
+                <updateRateHZ>100.0</updateRateHZ>
+                <gaussianNoise>0.0</gaussianNoise>
+                <frameName>imu_link</frameName>
                 <xyzOffset>0 0 0</xyzOffset>
                 <rpyOffset>0 0 0</rpyOffset>
-                <queueSize>${queueSize}</queueSize>
+                <queueSize>100</queueSize>
             </plugin>
             <pose>0 0 0 0 0 0</pose>
@@ -271,6 +252,6 @@
       <sensor type="ray" name="livox_mid360">
         <pose>0 0 0 0 0 0</pose>
-        <visualize>${visualize}</visualize>
-        <update_rate>${update_rate}</update_rate>
+        <visualize>false</visualize>
+        <update_rate>10</update_rate>
         <!-- This ray plugin is only for visualization. -->
         <plugin name="gazebo_ros_laser_controller" filename="liblivox_laser_simulation.so">
@@ -278,31 +259,33 @@
                 <scan>
                   <horizontal>
-                    <samples>0</samples>
+                    <samples>100</samples>
                     <resolution>1</resolution>
-                    <min_angle>${0}</min_angle>
-                    <max_angle>${2*PI}</max_angle>
+                    <min_angle>${-PI}</min_angle>
+                    <max_angle>${PI}</max_angle>
                   </horizontal>
                   <vertical>
-                    <samples>0</samples>
+                    <samples>50</samples>
                     <resolution>1</resolution>
-                    <min_angle>${-7.22/180*PI}</min_angle>
-                    <max_angle>${55.22/180*PI}</max_angle>
+                    <min_angle>${-PI}</min_angle>
+                    <max_angle>${PI}</max_angle>
                   </vertical>
                 </scan>
                 <range>
-                  <min>${laser_min_range}</min>
-                  <max>${laser_max_range}</max>
-                  <resolution>${resolution}</resolution>
+                  <min>0.1</min>
+                  <max>40</max>
+                  <resolution>1</resolution>
                 </range>
                 <noise>
                   <type>gaussian</type>
-                  <mean>${noise_mean}</mean>
-                  <stddev>${noise_stddev}</stddev>
+                  <mean>0.0</mean>
+                  <stddev>0.0</stddev>
                 </noise>
             </ray>
-            <samples>${samples}</samples>
-    	    <downsample>${downsample}</downsample>
+            <visualize>True</visualize>
+            <samples>20000</samples>
+    	    <downsample>1</downsample>
     	    <csv_file_name>mid360.csv</csv_file_name>
-    	    <ros_topic>${ros_topic}</ros_topic>
+    	    <ros_topic>/livox/lidar</ros_topic>
+            <publish_pointcloud_type>3</publish_pointcloud_type>
             <broadcastTF>false</broadcastTF>
         </plugin>

Commit message: update readme add new planner

File: src/sentry_simulation/urdf/main.urdf.xacro (robot description, xacro)
@@ -8,16 +8,16 @@
         <visual>
             <geometry>
-                    <cylinder length="0.05" radius="0.18" />
+                    <cylinder length="0.05" radius="0.1" />
             </geometry>
-            <origin rpy="0 0 1.57075" xyz="0 0 0.07" />
+            <origin rpy="0 0 1.57075" xyz="0 0 0.01" />
             <material name="White" />
         </visual>
         <collision>
             <geometry>
-                    <cylinder length="0.005" radius="0.15" />
+                    <cylinder length="0.005" radius="0.2" />
             </geometry>
-            <origin rpy="0 0 1.57075" xyz="0 0 0.07" />
+            <origin rpy="0 0 1.57075" xyz="0 0 0.01" />
         </collision>
-        <xacro:cylinder_inertial_matrix m="250" r="0.18" h="0.05" />
+        <xacro:cylinder_inertial_matrix m="10" r="0.1" h="0.05" />
     </link>
     <gazebo reference="base_link">
@@ -26,14 +26,14 @@
     </gazebo>
     <xacro:wheel_macro name="1" color="Red"
-                       xyz="0.2 -0.2 0.0326524329692152"
-                       rpy="-1.5707963267949 -6.12303176911189E-17 -2.35619445" />
+                       xyz="0.1 -0.1 0.0099524329692152"
+                       rpy="1.5707963267949 -6.12303176911189E-17 -2.35619445" />
+    <xacro:wheel_macro name="3" color="Black"
+                       xyz="-0.1 0.1 0.0099524329692152"
+                       rpy="1.5707963267949 3.06151588454563E-17 0.78539815" />
     <xacro:wheel_macro name="2" color="Blue"
-                       xyz="-0.2 0.2 0.0326524329692152"
-                       rpy="1.5707963267949 3.06151588454563E-17 0.78539815" />
-    <xacro:wheel_macro name="3" color="Black"
-                       xyz="0.2 0.2 0.0326524329692152"
+                       xyz="0.1 0.1 0.0099524329692152"
                        rpy="1.57079632679490 3.06151588456647E-17 -0.78539815" />
     <xacro:wheel_macro name="4" color="Green"
-                       xyz="-0.2 -0.2 0.0326524329692152"
+                       xyz="-0.1 -0.1 0.0099524329692152"
                        rpy="1.5707963267949 3.06151588456647E-17 2.35619445" />
     <!-- //// ////////////////////////////// driver controller ///////////////////  -->
@@ -53,3 +53,8 @@
         </plugin>
     </gazebo>
+	<!-- <gazebo>
+		<plugin name="gazebo_ros_control" filename="libgazebo_ros_control.so">
+		<robotNamespace></robotNamespace>
+		</plugin>
+	</gazebo> -->
 </robot>

File: src/sentry_simulation/urdf/sensor.urdf.xacro (robot description, xacro)
@@ -108,5 +108,5 @@
             </ray>
             <visualize>false</visualize>
-            <samples>20000</samples>
+            <samples>50000</samples>
     	    <downsample>1</downsample>
     	    <csv_file_name>mid360.csv</csv_file_name>

File: src/sentry_simulation/urdf/wheel.urdf.xacro (robot description, xacro)
@@ -28,6 +28,16 @@
             <parent link="base_link" />
             <child link="wheel_${name}_link" />
-            <axis xyz="0 0 0" />
+            <axis xyz="0 0 1" />
         </joint>
+		<transmission name="wheel_${name}_transmission">
+			<type>transmission_interface/SimpleTransmission</type>
+			<joint name="wheel_${name}_joint">
+				<hardwareInterface>hardware_interface/VelocityJointInterface</hardwareInterface>
+			</joint>
+			<actuator name="wheel_${name}_motor">
+				<hardwareInterface>hardware_interface/VelocityJointInterface</hardwareInterface>
+				<mechanicalReduction>1</mechanicalReduction>
+			</actuator>
+		</transmission>
         <gazebo reference="wheel_${name}_link">
             <pose>0 0 0 0 0 0</pose>

Commit message: update readme and fix the abnormal pointcloud

File: src/sentry_simulation/urdf/main.urdf.xacro (robot description, xacro)
@@ -47,4 +47,8 @@
             <odometryRate>10.0</odometryRate>
             <odometryFrame>gazebo_odom</odometryFrame>
+            <!-- <leftFrontJoint>wheel_2_joint</leftFrontJoint>
+            <rightFrontJoint>wheel_1_joint</rightFrontJoint>
+            <leftRearJoint>wheel_3_joint</leftRearJoint>
+            <rightRearJoint>wheel_4_joint</rightRearJoint> -->
             <robotBaseFrame>gazebo_base_link</robotBaseFrame>
             <cmdTimeout>3.0</cmdTimeout>
@@ -53,8 +57,3 @@
         </plugin>
     </gazebo>
-	<!-- <gazebo>
-		<plugin name="gazebo_ros_control" filename="libgazebo_ros_control.so">
-		<robotNamespace></robotNamespace>
-		</plugin>
-	</gazebo> -->
 </robot>

File: src/sentry_simulation/urdf/sensor.urdf.xacro (robot description, xacro)
@@ -26,17 +26,10 @@
     <link name="livox_mid360">
         <visual>
-            <origin xyz="0 0 0" rpy="0 0 0" />
+            <origin xyz="0 0 0" rpy="${PI/2} 0 ${PI}" />
             <geometry>
-                <mesh filename="package://sentry_simulation/mesh/mid360.stl">
+                <mesh filename="package://sentry_simulation/mesh/mid360.stl" scale="0.0008 0.0008 0.0008">
                 </mesh>
             </geometry>
        </visual>
-        <collision>
-            <origin xyz="0 0 0" rpy="0 0 0" />
-            <geometry>
-                <mesh filename="package://sentry_simulation/mesh/mid360.stl">
-                </mesh>
-            </geometry>
-        </collision>
     </link>
    <joint name="imu_joint" type="fixed">
@@ -98,5 +91,5 @@
                 <range>
                   <min>0.1</min>
-                  <max>40</max>
+                  <max>40.0</max>
                   <resolution>1</resolution>
                 </range>
@@ -107,6 +100,6 @@
                 </noise>
             </ray>
-            <visualize>false</visualize>
-            <samples>50000</samples>
+            <visualize>true</visualize>
+            <samples>20000</samples>
     	    <downsample>1</downsample>
     	    <csv_file_name>mid360.csv</csv_file_name>

File: src/sentry_simulation/urdf/wheel.urdf.xacro (robot description, xacro)
@@ -29,6 +29,7 @@
             <child link="wheel_${name}_link" />
             <axis xyz="0 0 1" />
+            <limit effort="30" velocity="17.4" />
         </joint>
-		<transmission name="wheel_${name}_transmission">
+		<!-- <transmission name="wheel_${name}_transmission">
 			<type>transmission_interface/SimpleTransmission</type>
 			<joint name="wheel_${name}_joint">
@@ -39,6 +40,12 @@
 				<mechanicalReduction>1</mechanicalReduction>
 			</actuator>
-		</transmission>
+		</transmission> -->
         <gazebo reference="wheel_${name}_link">
+            <mu1>0</mu1>
+            <mu2>0</mu2>
+            <kp>200000.0</kp>
+            <kd>10.0</kd>
+            <minDepth>0.001</minDepth>
+            <maxVel>1.0</maxVel>
             <pose>0 0 0 0 0 0</pose>
             <material>Gazebo/${color}</material>

Commit message: add mbf

File: src/sentry_simulation/urdf/main.urdf.xacro (robot description, xacro)
@@ -8,5 +8,5 @@
         <visual>
             <geometry>
-                    <cylinder length="0.05" radius="0.1" />
+                    <cylinder length="0.05" radius="0.25" />
             </geometry>
             <origin rpy="0 0 1.57075" xyz="0 0 0.01" />
@@ -15,9 +15,9 @@
         <collision>
             <geometry>
-                    <cylinder length="0.005" radius="0.2" />
+                    <cylinder length="0.005" radius="0.25" />
             </geometry>
             <origin rpy="0 0 1.57075" xyz="0 0 0.01" />
         </collision>
-        <xacro:cylinder_inertial_matrix m="10" r="0.1" h="0.05" />
+        <xacro:cylinder_inertial_matrix m="80" r="0.1" h="0.05" />
     </link>
     <gazebo reference="base_link">
@@ -42,6 +42,5 @@
             <robotNamespace>/</robotNamespace>
             <commandTopic>/cmd_vel</commandTopic>
-            <!-- 因为关闭发布odom的tf没有效果，所以此处把parent link改为gazebo_odom,child link改为gazebo_base_link
-            仍可以通过cmd_vel话题来控制小车的运动，同时可以跑其他里程计算法，避免干扰 -->
+            <!-- set the publish rate 0.0 hz to close the odometry -->
             <odometryRate>0.0</odometryRate>
             <odometryTopic>/gazebo_odom</odometryTopic>

File: src/sentry_simulation/urdf/sensor.urdf.xacro (robot description, xacro)
@@ -71,5 +71,5 @@
       <sensor type="ray" name="livox_mid360">
         <pose>0 0 0 0 0 0</pose>
-        <visualize>true</visualize>
+        <visualize>True</visualize>
         <update_rate>10</update_rate>
         <plugin name="gazebo_ros_laser_controller" filename="liblivox_laser_simulation.so">
@@ -100,5 +100,5 @@
                 </noise>
             </ray>
-            <visualize>fasle</visualize>
+            <visualize>Fasle</visualize>
             <samples>20000</samples>
     	    <downsample>1</downsample>
@@ -106,5 +106,5 @@
     	    <ros_topic>/livox/lidar</ros_topic>
             <publish_pointcloud_type>3</publish_pointcloud_type>
-            <broadcastTF>false</broadcastTF>
+            <!-- <broadcastTF>Fasle</broadcastTF> -->
         </plugin>
       </sensor>
