Commit message: add the normal scqn and livoxmsgs convert

File: src/sentry_simulation/sentry_description/urdf/sensor.urdf.xacro (robot description, xacro)
@@ -24,5 +24,5 @@
         </inertial>
     </link>
-    <link name="livox_mid360">
+    <link name="livox_frame">
         <visual>
             <origin xyz="0 0 0" rpy="${PI/2} 0 ${PI}" />
@@ -41,5 +41,5 @@
     <joint name="base_lidar" type="fixed">
         <parent link="base_link" />
-        <child link="livox_mid360" />
+        <child link="livox_frame" />
         <origin xyz="0.135 0 0.08" rpy="0 0 0" />
     </joint>
@@ -68,6 +68,6 @@
     </gazebo>
     <!-- //////////////////////////////// lidar control ////////////////////////////////// -->
-    <gazebo reference="livox_mid360">
-      <sensor type="ray" name="livox_mid360">
+    <gazebo reference="livox_frame">
+      <sensor type="ray" name="livox_frame">
         <pose>0 0 0 0 0 0</pose>
         <visualize>True</visualize>
